File: STM32_Board_Bluetooth_v1.kicad_sch (KiCad schematic)
At the start: 42 parts, among them J101 Conn_01x04, J102 USB_C_Receptacle_USB2.0_16P, J103 Conn_Coaxial, J104 TC2030, SW101 SW_Push, U101 MIC5365-3.3YD5, U102 STM32WB55CEU6, Y101 32MHz, Y102 32kHz768

Commit message: Add files via upload
Parts:
- C101, C110, C111, C112, C115: footprint (none) -> Capacitor_SMD:C_0603_1608Metric
- C102, C103, C104, C105, C106, C107, C108, C109, C113, C114, C116, C117, C118: footprint (none) -> Capacitor_SMD:C_0402_1005Metric
- C119, C120: value C -> 10p; footprint (none) -> Capacitor_SMD:C_0402_1005Metric
- D101: footprint (none) -> LED_SMD:LED_0402_1005Metric
- J101: footprint (none) -> Connector_Molex:Molex_PicoBlade_53048-0410_1x04_P1.25mm_Horizontal
- J102: footprint (none) -> Connector_USB:USB_C_Receptacle_GCT_USB4105-xx-A_16P_TopMnt_Horizontal
- J103: footprint (none) -> Connector_Coaxial:U.FL_Hirose_U.FL-R-SMT-1_Vertical
- L101: footprint (none) -> Inductor_SMD:L_0805_2012Metric
- L102, L103: footprint (none) -> Inductor_SMD:L_0402_1005Metric
- R101, R102, R103, R104, R105, R106, R107: footprint (none) -> Resistor_SMD:R_0402_1005Metric
- SW101: footprint (none) -> Button_Switch_SMD:SW_SPST_CK_RS282G05A3
- Y101: footprint (none) -> Crystal:Crystal_SMD_2016-4Pin_2.0x1.6mm
- Y102: footprint (none) -> Crystal:Crystal_SMD_2012-2Pin_2.0x1.2mm
Connections:
- net USB_CC2: now reaches J102.B5 (CC2), R105.1
- net USBC_D-: now reaches J102.A7 (D-), J102.B7 (D-), Ude101.1 (I/O1)
- net USBC_D+: now reaches J102.A6 (D+), J102.B6 (D+), Ude101.3 (I/O2)
- net USB_CC1: now reaches J102.A5 (CC1), R104.1
Other:
- note added: "Video #114 for more detail in hardware design"
- note removed: "1:48:15"
- moved on the sheet: R104
